Commit message: feat: añadir ros2_control para mover el robot en simulación
- Añadir bloque ros2_control con plugin gz_ros2_control en URDF
- Crear archivo de configuración wx250_controllers.yaml
- Cargar joint_state_broadcaster, arm_controller y gripper_controller
- Añadir bridge del clock para sincronización con tiempo de simulación
- Robot ahora se mueve correctamente con comandos JointTrajectory

File: sim_gazebo/urdf/wx250_gz.urdf.xacro (robot description, xacro)
@@ -34,3 +34,65 @@
     </plugin>
   </gazebo>
+  <!-- Sobrescribir ros2_control para usar gz_ros2_control en simulación -->
+  <ros2_control name="GazeboSystem" type="system">
+    <hardware>
+      <plugin>gz_ros2_control/GazeboSimSystem</plugin>
+    </hardware>
+    <joint name="waist">
+      <command_interface name="position">
+        <param name="min">-3.14</param>
+        <param name="max">3.14</param>
+      </command_interface>
+      <state_interface name="position"/>
+      <state_interface name="velocity"/>
+    </joint>
+    <joint name="shoulder">
+      <command_interface name="position">
+        <param name="min">-1.88</param>
+        <param name="max">1.99</param>
+      </command_interface>
+      <state_interface name="position"/>
+      <state_interface name="velocity"/>
+    </joint>
+    <joint name="elbow">
+      <command_interface name="position">
+        <param name="min">-2.15</param>
+        <param name="max">1.61</param>
+      </command_interface>
+      <state_interface name="position"/>
+      <state_interface name="velocity"/>
+    </joint>
+    <joint name="wrist_angle">
+      <command_interface name="position">
+        <param name="min">-1.75</param>
+        <param name="max">2.15</param>
+      </command_interface>
+      <state_interface name="position"/>
+      <state_interface name="velocity"/>
+    </joint>
+    <joint name="wrist_rotate">
+      <command_interface name="position">
+        <param name="min">-3.14</param>
+        <param name="max">3.14</param>
+      </command_interface>
+      <state_interface name="position"/>
+      <state_interface name="velocity"/>
+    </joint>
+    <joint name="left_finger">
+      <command_interface name="position">
+        <param name="min">0.015</param>
+        <param name="max">0.037</param>
+      </command_interface>
+      <state_interface name="position"/>
+      <state_interface name="velocity"/>
+    </joint>
+  </ros2_control>
+  <!-- Plugin de gz_ros2_control para Gazebo Harmonic -->
+  <gazebo>
+    <plugin
+      filename="gz_ros2_control-system"
+      name="gz_ros2_control::GazeboSimROS2ControlPlugin">
+      <parameters>$(find sim_gazebo)/config/wx250_controllers.yaml</parameters>
+    </plugin>
+  </gazebo>
 </robot>

Commit message: feat: anclaje robot a plataforma + vasos huecos + use_sim_time
- Anclaje físico robot mediante joint fijo en URDF (link world + world_fixed)
- Eliminado spawn dinámico con coordenadas (ahora viene del URDF)
- Eliminado static_tf_world_robot redundante
- ParameterValue para evitar error de parsing de robot_description
- Nuevo launch arm_robot.launch.py con use_sim_time=True
- Vasos modelados como cilindros huecos (12 paredes + fondo)
- Vasos con colores llamativos para mejorar detección

File: sim_gazebo/urdf/wx250_gz.urdf.xacro (robot description, xacro)
@@ -9,4 +9,11 @@
   <!-- Incluir el URDF original del WX250 -->
   <xacro:include filename="$(find interbotix_xsarm_descriptions)/urdf/wx250.urdf.xacro"/>
+  <!-- Joint fijo world→base_link: ancla físicamente el robot al mundo en Gazebo Harmonic -->
+  <link name="world"/>
+  <joint name="world_fixed" type="fixed">
+    <origin xyz="-0.165 0 0.4" rpy="0 0 0"/>
+    <parent link="world"/>
+    <child link="wx250/base_link"/>
+  </joint>
   <!-- Añadir materiales/colores para visualización en Gazebo -->
   <gazebo reference="wx250/base_link">
@@ -96,3 +103,7 @@
     </plugin>
   </gazebo>
+  <gazebo>
+    <static>false</static>
+    <self_collide>false</self_collide>
+  </gazebo>
 </robot>

Commit message: feat: gripper funcional con mimic joint en gz_ros2_control
- Mesa bajada a z=0.30 para mejor margen vertical
- Vasos reposicionados a z=0.30
- right_finger configurado con mimic en ros2_control (no en física dartsim)
- gz_ros2_control aplica el mimic a nivel de controlador
- Ambos dedos del gripper se cierran sincronizados al ejecutar gripper_close()

File: sim_gazebo/urdf/wx250_gz.urdf.xacro (robot description, xacro)
@@ -102,4 +102,10 @@
       <state_interface name="velocity"/>
     </joint>
+    <joint name="right_finger">
+      <param name="mimic">left_finger</param>
+      <param name="multiplier">-1.0</param>
+      <state_interface name="position"/>
+      <state_interface name="velocity"/>
+    </joint>
   </ros2_control>
   <!-- Plugin de gz_ros2_control para Gazebo Harmonic -->
